Commit message: change robot model

File: robots/xiaoqiang_udrf.URDF (robot description, URDF)
Before this commit: robot xiaoqiang_udrf, 4 links, 3 joints
Links:
- added link kinect_Link, mass 0.669252371670692; collision mesh filename=package://xiaoqiang_udrf/meshes/kinect_Link.STL; visual mesh filename=package://xiaoqiang_udrf/meshes/kinect_Link.STL
- added link lidar_link, mass 0.0984481070530837; collision mesh filename=package://xiaoqiang_udrf/meshes/lidar_link.STL; visual mesh filename=package://xiaoqiang_udrf/meshes/lidar_link.STL
- link back_wheel: mass 0.070437 -> 0.0646530070020808
- link base_link: mass 4.3093 -> 4.77346929236529
- link left_wheel: mass 0.4651 -> 0.18816486485113
- link right_wheel: mass 0.4651 -> 0.188164864851131
Joints:
- added joint fix1: type fixed, parent base_link, child kinect_Link, origin xyz=-0.135557187224918 -0.000112698372204401 0.255 rpy=-1.57079632679489 0 -1.5707963267949, axis 0 0 0
- added joint rot4: type continuous, parent base_link, child lidar_link, origin xyz=-0.258786796564404 6.46265772448196E-05 0.305000000000001 rpy=-1.5707963267949 -3.15213658012586E-15 -0.452067123629806, axis 0 1 0
- joint rot1: origin xyz=0 -0.176 -0.05489 rpy=1.5708 0 0 -> xyz=0 -0.150112698372207 -0.06 rpy=1.57079632679477 1.52790873038023 -1.29473733419683E-13
- joint rot2: axis 0 0 -1 -> 0 0 1; origin xyz=0 0.176 -0.05489 rpy=-1.5708 0 3.1416 -> xyz=0 0.149887301627792 -0.0599999999999983 rpy=-1.5707963267949 0.357463595053736 1.22790071016839E-29
- joint rot3: origin xyz=-0.25204 -0.00060998 -0.037 rpy=1.5708 0 -5.9631E-17 -> xyz=-0.278786796564403 -0.000112698372207953 -0.046000000000001 rpy=1.5707963267949 -3.45895916116442E-15 -0.160759229830102

Commit message: change xiaoqiang mini model

File: robots/xiaoqiang_udrf.URDF (robot description, URDF)
Before this commit: robot xiaoqiang_udrf, 6 links, 5 joints
Links:
- removed link kinect_Link
- added link kinect_link, mass 0.588695422153955; collision mesh filename=package://xiaoqiang_udrf/meshes/kinect_link.STL; visual mesh filename=package://xiaoqiang_udrf/meshes/kinect_link.STL
- link back_wheel: mass 0.0646530070020808 -> 0.0646530057023567
- link base_link: mass 4.77346929236529 -> 2.67497367621507
- link left_wheel: mass 0.18816486485113 -> 0.188164864851131
- link lidar_link: mass 0.0984481070530837 -> 0.0984481070530836
Joints:
- removed joint fix1
- added joint rot5: type continuous, parent base_link, child lidar_link, origin xyz=-0.18 0 0.21 rpy=-1.5708 -4.5495E-17 2.4485, axis 0 1 0
- joint rot1: origin xyz=0 -0.150112698372207 -0.06 rpy=1.57079632679477 1.52790873038023 -1.29473733419683E-13 -> xyz=0 -0.105 -0.04 rpy=-1.5708 0.98189 -3.1416
- joint rot2: origin xyz=0 0.149887301627792 -0.0599999999999983 rpy=-1.5707963267949 0.357463595053736 1.22790071016839E-29 -> xyz=0 0.105 -0.04 rpy=1.5708 -1.1924 -3.1416
- joint rot3: origin xyz=-0.278786796564403 -0.000112698372207953 -0.046000000000001 rpy=1.5707963267949 -3.45895916116442E-15 -0.160759229830102 -> xyz=-0.145 0 -0.026 rpy=1.5708 6.7329E-18 -0.09469
- joint rot4: axis 0 1 0 -> -1 0 0; child lidar_link -> kinect_link; limit (none) -> lower=-0.3 upper=0.3 effort=10 velocity=10; origin xyz=-0.258786796564404 6.46265772448196E-05 0.305000000000001 rpy=-1.5707963267949 -3.15213658012586E-15 -0.452067123629806 -> xyz=-0.11677 0 0.16 rpy=-1.6034 7.1211E-17 -1.5708; type continuous -> revolute

Commit message: change kinect_link name

File: robots/xiaoqiang_udrf.URDF (robot description, URDF)
Before this commit: robot xiaoqiang_udrf, 6 links, 5 joints
Links:
- removed link kinect_link
- added link kinect_link1, mass 0.588695422153955; collision mesh filename=package://xiaoqiang_udrf/meshes/kinect_link.STL; visual mesh filename=package://xiaoqiang_udrf/meshes/kinect_link.STL
Joints:
- joint rot4: child kinect_link -> kinect_link1
