Commit message: add lungu branch

File: robots/xiaoqiang_udrf.urdf (robot description, URDF)
Before this commit: robot xiaoqiang_udrf, 6 links, 5 joints
Links:
- removed link back_wheel
- removed link kinect_Link
- added link front1_wheel, mass 0.126682636045453; collision mesh filename=package://xiaoqiang_udrf/meshes/front1_wheel.STL; visual mesh filename=package://xiaoqiang_udrf/meshes/front1_wheel.STL
- added link front2_wheel, mass 0.126682635871512; collision mesh filename=package://xiaoqiang_udrf/meshes/front2_wheel.STL; visual mesh filename=package://xiaoqiang_udrf/meshes/front2_wheel.STL
- added link kinect_link, mass 0.588695418123486; collision mesh filename=package://xiaoqiang_udrf/meshes/kinect_link.STL; visual mesh filename=package://xiaoqiang_udrf/meshes/kinect_link.STL
- link base_link: mass 4.77346929236529 -> 8.36303567682231
- link left_wheel: mass 0.18816486485113 -> 0.834069618273221
- link lidar_link: mass 0.0984481070530837 -> 0.0984481791975763
- link right_wheel: mass 0.188164864851131 -> 0.834069618273221
Joints:
- removed joint fix1
- removed joint rot1
- removed joint rot2
- removed joint rot3
- removed joint rot4
- added joint kinect: type continuous, parent base_link, child kinect_link, origin xyz=0.13823 0 0.255 rpy=-1.4803 0 -1.5708, axis 1 0 0
- added joint left_rot: type continuous, parent base_link, child front1_wheel, origin xyz=0.26879 0.0795 -0.02225 rpy=1.5708 0 -2.0971, axis 0 1 0
- added joint left_whell: type continuous, parent base_link, child left_wheel, origin xyz=0 0.137 -0.035 rpy=-1.5708 0.68527 -3.1416, axis 0 0 1
- added joint lidar: type continuous, parent base_link, child lidar_link, origin xyz=-0.015 0.00017732 0.335 rpy=-1.5708 1.7959E-17 -1.2422, axis 0 -1 0
- added joint right_rot: type continuous, parent base_link, child front2_wheel, origin xyz=0.26879 -0.0805 -0.02225 rpy=1.5708 0 -0.38246, axis 0 1 0
- added joint right_wheel: type continuous, parent base_link, child right_wheel, origin xyz=0 -0.137 -0.035 rpy=-1.5708 0.82165 5.3376E-17, axis 0 0 -1

Commit message: rename kinect_link

File: robots/xiaoqiang_udrf.urdf (robot description, URDF)
Before this commit: robot xiaoqiang_udrf, 7 links, 6 joints
Links:
- removed link kinect_link
- added link kinect_Link, mass 0.588695418123486; collision mesh filename=package://xiaoqiang_udrf/meshes/kinect_link.STL; visual mesh filename=package://xiaoqiang_udrf/meshes/kinect_link.STL
Joints:
- joint kinect: child kinect_link -> kinect_Link

Commit message: 赤兔基础模型包

File: robots/xiaoqiang_udrf.urdf (robot description, URDF)
Before this commit: robot xiaoqiang_udrf, 7 links, 6 joints
Links:
- removed link front1_wheel
- removed link front2_wheel
- removed link kinect_Link
- removed link lidar_link
- added link back_wheel1, mass 0.134574489008056; collision mesh filename=package://xiaoqiang_udrf/meshes/back_wheel1.STL; visual mesh filename=package://xiaoqiang_udrf/meshes/back_wheel1.STL
- added link back_wheel2, mass 0.134574489008056; collision mesh filename=package://xiaoqiang_udrf/meshes/back_wheel2.STL; visual mesh filename=package://xiaoqiang_udrf/meshes/back_wheel2.STL
- added link base_Link2, mass 0.112344913941376; collision mesh filename=package://xiaoqiang_udrf/meshes/base_Link2.STL; visual mesh filename=package://xiaoqiang_udrf/meshes/base_Link2.STL
- added link front_wheel1, mass 0.134574489008056; collision mesh filename=package://xiaoqiang_udrf/meshes/front_wheel1.STL; visual mesh filename=package://xiaoqiang_udrf/meshes/front_wheel1.STL
- added link front_wheel2, mass 0.134574489008056; collision mesh filename=package://xiaoqiang_udrf/meshes/front_wheel2.STL; visual mesh filename=package://xiaoqiang_udrf/meshes/front_wheel2.STL
- link base_link: mass 8.36303567682231 -> 5.51934540138491
- link left_wheel: mass 0.834069618273221 -> 0.804868654069467
- link right_wheel: mass 0.834069618273221 -> 0.804868654069467
Joints:
- removed joint kinect
- removed joint left_rot
- removed joint left_whell
- removed joint lidar
- removed joint right_rot
- removed joint right_wheel
- added joint rot1: type continuous, parent base_link, child left_wheel, origin xyz=0 0.1595 -0.023 rpy=1.5707963267949 1.5707963267949 0, axis 0 0 -1
- added joint rot2: type continuous, parent base_link, child right_wheel, origin xyz=0 -0.1595 -0.023 rpy=1.5707963267949 -1.49170041722774 3.14159265358979, axis 0 0 1
- added joint rot3: type continuous, parent base_link, child front_wheel1, origin xyz=0.175 0.135 -0.00500000000000002 rpy=1.5707963267949 0 0, axis 0 1 0
- added joint rot4: type continuous, parent base_link, child front_wheel2, origin xyz=0.175 -0.135 -0.005 rpy=1.5707963267949 0 0, axis 0 1 0
- added joint rot5: type continuous, parent base_link, child back_wheel1, origin xyz=-0.175 0.135 -0.00500000000000002 rpy=1.5707963267949 0 0, axis 0 1 0
- added joint rot6: type continuous, parent base_link, child back_wheel2, origin xyz=-0.175 -0.135 -0.005 rpy=1.5707963267949 0 0, axis 0 1 0
- added joint rot7: type fixed, parent base_link, child base_Link2, origin xyz=0 0 -0.08 rpy=0 0 1.5707963267949, axis 0 0 0
